File: DS100M06V_linear.kicad_pcb (KiCad board)
At the start: 4 copper layers, 100 x 60 mm, 140 parts, among them J1 wire2board, J10 BNC_panel_mount, J11 wire2board, J2 Wire2Board, J3 wire2board, J4 wire2board, J5 Wire2Board, J6 Wire2Board, J7 Wire2Board, J8 red_safety_4mm_connector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

Commit message: Ferrites.
Parts:
- added FB1: FerriteBead, Inductor_SMD:L_0603_1608Metric_Pad1.05x0.95mm_HandSolder, F.Cu at (123.9, 126.8)
- added FB2: FerriteBead, Inductor_SMD:L_0603_1608Metric_Pad1.05x0.95mm_HandSolder, F.Cu at (118.3, 125.5)
- added FB3: FerriteBead, Inductor_SMD:L_0603_1608Metric_Pad1.05x0.95mm_HandSolder, F.Cu at (150.3, 121.0)
- added FB4: FerriteBead, Inductor_SMD:L_0603_1608Metric_Pad1.05x0.95mm_HandSolder, F.Cu at (151.8, 111.9)
- moved R51 2.48 mm to (119.0, 127.3)
- moved TP4 0.36 mm to (167.0, 112.6)
- moved R18 0.10 mm to (148.5, 112.8)
Connections:
- C18 pad 2: -5V -> Net-(U1C-V-)
- C19 pad 2: +5V -> Net-(U1C-V+)
- C21 pad 2: +5V -> Net-(U4-V+)
- C22 pad 2: -5V -> Net-(U4-V-)
- C25 pad 2: -5V -> Net-(U4-V-)
- C26 pad 2: +5V -> Net-(U4-V+)
- C27 pad 2: -5V -> Net-(U1C-V-)
- C33 pad 2: +5V -> Net-(U1C-V+)
- C34 pad 2: +5V -> Net-(U1C-V+)
- C35 pad 2: -5V -> Net-(U1C-V-)
- C37 pad 2: +5V -> Net-(U4-V+)
- C38 pad 2: -5V -> Net-(U4-V-)
- U1 pad 4: -5V -> Net-(U1C-V-)
- U1 pad 8: +5V -> Net-(U1C-V+)
- U4 pad 4: -5V -> Net-(U4-V-)
- U4 pad 7: +5V -> Net-(U4-V+)
Routing:
- net +5V: track 153.2 -> 137.4 mm, vias 7 -> 4
- net Net-(U1C-V+): track 0.00 -> 11.3 mm
- net -5V: track 129.4 -> 119.8 mm, vias 8 -> 6
- net Net-(U4-V+): track 0.00 -> 7.61 mm
- net Net-(U1C-V-): track 0.00 -> 6.84 mm
- net Net-(U4-V-): track 0.00 -> 6.82 mm
- net Net-(U1A-+): track 8.45 -> 7.94 mm
