File: DS100M08KV.kicad_pcb (KiCad board)
At the start: 4 copper layers, 100 x 60 mm, 144 parts, among them J1 wire2board, J10 BNC_panel_mount, J11 wire2board, J2 Wire2Board, J3 wire2board, J4 wire2board, J5 Wire2Board, J6 Wire2Board, J7 Wire2Board, J8 red_safety_4mm_connector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

Commit message: Cleaning up libraries.
Parts:
- removed H10, H11, H12, H13, H14, H15, H16, H17, H18, H19, H20, H9: MountingHole, MountingHole:MountingHole_3.2mm_M3
- J10: footprint DS100M06V_linear:BNC_panel_mount -> DS100M08KV:BNC_panel_mount
- J8: footprint DS100M06V_linear:red_safety_4mm_connector -> DS100M08KV:red_safety_4mm_connector
- J9: footprint DS100M06V_linear:red_safety_4mm_connector -> DS100M08KV:black_safety_4mm_connector
- SW1, SW2: footprint DS100M06V_linear:DPDT_bigger -> DS100M08KV:DPDT_bigger
Routing:
- net (no net): vias 168 -> 0
Other:
- board size 100 x 60 mm -> 100 x 52 mm

Commit message: Housekeeping.
Parts:
- removed H5, H6, H7, H8: WireFeedHole, MountingHole:MountingHole_2.2mm_M2_ISO7380
- removed L1: 4.7u, Inductor_SMD:L_Bourns_SRN6045TA
- added L3: 4.7u, Inductor_SMD:L_Bourns_SRN6045TA, F.Cu at (157.4, 139.8)
- moved R26 8.91 mm to (147.8, 148.2), turned to 180 degrees
- moved R21 3.64 mm to (144.0, 148.2), turned to 180 degrees
- moved R25 0.25 mm to (150.6, 142.8)
Connections:
- U2 pad 1: (no net) -> Net-(U2-TEMP)
- U2 pad 6: Net-(U2-TEMP) -> unconnected-(U2-~{STDBY}-Pad6)
- U2 pad 7: (no net) -> unconnected-(U2-~{CHRG}-Pad7)
Routing:
- net Net-(U2-TEMP): track 4.23 -> 5.95 mm
- net +VBUS: track 5.99 -> 7.64 mm
- net Earth: track 18.0 -> 18.8 mm

Commit message: Clearer
Parts:
- removed J2, J5: Wire2Board, Connector_Wire:SolderWire-0.127sqmm_1x01_D0.48mm_OD1mm
- added J12: Conn_01x04_Socket, Connector_JST:JST_PH_B4B-PH-K_1x04_P2.00mm_Vertical, B.Cu at (126.5, 146.6)
- RV2: moved to B.Cu
- moved SW1 4.35 mm to (132.5, 117.2)
- moved SW2 4.35 mm to (132.5, 132.8)
- moved H3 2.70 mm to (100.0, 142.3)
- moved H4 2.60 mm to (180.0, 142.3)
- moved H2 2.40 mm to (180.0, 107.3)
- moved H1 2.30 mm to (100.0, 107.3)
- moved C40 2.26 mm to (169.4, 145.1), turned to 180 degrees
Routing:
- net +VBUS: track 7.64 -> 20.3 mm
- net Net-(PS1-+Vin): track 52.2 -> 49.8 mm
Other:
- board text added: "+"
- board text added: "-"

Commit message: small updates.
Parts:
- turned R6 to -90 degrees
Changed lines of the file:
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@@
 	(footprint "Resistor_SMD:R_0603_1608Metric_Pad0.98x0.95mm_HandSolder"
 		(layer "F.Cu")
-		(at 142.3 113.6 180)
+		(at 142.3 113.6 -90)
 		(descr "Resistor SMD 0603 (1608 Metric), square (rectangular) end terminal, IPC_7351 nominal with elongated pad for handsoldering. (Body size source: IPC-SM-782 page 72, https://www.pcb-3d.com/wordpress/wp-content/uploads/ipc-sm-782a_amendment_1_and_2.pdf), generated with kicad-footprint-generator")
 		(tags "resistor handsolder")
 		(property "Reference" "R6"
-			(at 0 -1.43 0)
+			(at 0 -1.43 90)
 			(layer "F.SilkS")
 			(hide yes)
@@
 		)
 		(property "Value" "50"
-			(at 0 1.43 0)
+			(at 0 1.43 90)
 			(layer "F.Fab")
 			(hide yes)
@@
 		)
 		(property "Datasheet" ""
-			(at 0 0 180)
+			(at 0 0 270)
 			(unlocked yes)
 			(layer "F.Fab")
@@
 		)
 		(property "Description" ""
-			(at 0 0 180)
+			(at 0 0 270)
 			(unlocked yes)
 			(layer "F.Fab")
@@
 		)
 		(fp_line
-			(start 1.65 0.73)
-			(end -1.65 0.73)
+			(start -1.65 0.73)
+			(end -1.65 -0.73)
 			(stroke
 				(width 0.05)
@@
 		)
 		(fp_line
-			(start 1.65 -0.73)
-			(end 1.65 0.73)
+			(start 1.65 0.73)
+			(end -1.65 0.73)
 			(stroke
 				(width 0.05)
@@
 		)
 		(fp_line
-			(start -1.65 0.73)
-			(end -1.65 -0.73)
+			(start -1.65 -0.73)
+			(end 1.65 -0.73)
 			(stroke
 				(width 0.05)
@@
 		)
 		(fp_line
-			(start -1.65 -0.73)
-			(end 1.65 -0.73)
+			(start 1.65 -0.73)
+			(end 1.65 0.73)
 			(stroke
 				(width 0.05)
@@
 		)
 		(fp_line
-			(start 0.8 0.4125)
-			(end -0.8 0.4125)
+			(start -0.8 0.4125)
+			(end -0.8 -0.4125)
 			(stroke
 				(width 0.1)
@@
 		)
 		(fp_line
-			(start 0.8 -0.4125)
-			(end 0.8 0.4125)
+			(start 0.8 0.4125)
+			(end -0.8 0.4125)
 			(stroke
 				(width 0.1)
@@
 		)
 		(fp_line
-			(start -0.8 0.4125)
-			(end -0.8 -0.4125)
+			(start -0.8 -0.4125)
+			(end 0.8 -0.4125)
 			(stroke
 				(width 0.1)
@@
 		)
 		(fp_line
-			(start -0.8 -0.4125)
-			(end 0.8 -0.4125)
+			(start 0.8 -0.4125)
+			(end 0.8 0.4125)
 			(stroke
 				(width 0.1)
@@
 		)
 		(pad "1" smd roundrect
-			(at -0.9125 0 180)
+			(at -0.9125 0 270)
 			(size 0.975 0.95)
 			(layers "F.Cu" "F.Mask" "F.Paste")
@@
 		)
 		(pad "2" smd roundrect
-			(at 0.9125 0 180)
+			(at 0.9125 0 270)
 			(size 0.975 0.95)
 			(layers "F.Cu" "F.Mask" "F.Paste")
@@
 			"AABRFgAAAAAAAJBpO0sAAAAAIHtfI0l/AAAAAAAAAAAAAAAAAAAAAAAAcgAAAAAAAAAhFgAAAAAA"
 			"AJBpO0sAAAAAIHtfI0l/AAAAAAAAAAAAAAAAAAAAAAAAwHg7SwAAAADxFQAAAAAAAJBpO0sAAAAA"
-			"IHtfI0l/AAAAAAAAAAAAAAAAAAAA"
+			"IHtfI0l/AAAAAAAAAAAAAAAAAAAAAAAAAAAAAAAAAABLogEAIAAAAEjsEBYAAAAAbAQAAHQAAAAA"
+			"AAAAAAAAAEuiAQA2AAAAaOwQFgAAAABZBAAAUwAAAAAAAAAAAAAAS6IBACwAAACI7BAWAAAAAFgE"
+			"AABCAAAAAAAAAAAAAABLogEAUAAAAKjsEBYAAAAAVwQAACwAAAAAAAAAAAAAAEuiAQBBAAAAyOwQ"
+			"FgAAAABPBAAAVAAAAAAAAAAAAAAAS6IBAC0AAADo7BAWAAAAAFIEAAAtAAAAAAAAAAAAAABLogEA"
+			"AAAAAAjtEBYAAAAAZgQAAAAAAADQ8xAWAAAAAFSiAQAyAAAAAAAAAAAAAABnBAAAYgAAANDzEBYA"
+			"AAAAVKIBAGEAAABI7RAWAAAAAGgEAAAgAAAA0PMQFgAAAABUogEAIAAAAGjtEBYAAAAAaQQAAHQA"
+			"AADQ8xAWAAAAAFSiAQA2AAAAiO0QFgAAAABqBAAAcwAAANDzEBYAAAAAVKIBACwAAACo7RAWAAAA"
+			"AGsEAABiAAAA0PMQFgAAAABUogEAcAAAAMjtEBYAAAAAbwQAACwAAADQ8xAWAAAAAFSiAQBhAAAA"
+			"6O0QFgAAAAAYAAAAdAAAALBl89IWfwAAAQAAAC0AAAA2AAAANAAAAPtPAAAPAAAA+08AABYAAAAY"
+			"AAAAAAAAACAf/tIWfwAAAQAAAGsAAABhAAAAZwAAAPtPAAAXAAAA+08AADYAAAAVAAAAOgAAACju"
+			"EBYAAAAAIB/+0hZ/AAABAAAANgAAAPtPAAAPAAAA+08AADYAAAAYAAAAMQAAACDrLw8XfwAAAQAA"
+			"AF8AAABwAAAAMAAAAPtPAAA3AAAA+08AADsAAABmBAAAAAAAAMjvEBYAAAAAUaIBAAAAAAAAAAAA"
+			"AAAAAGcEAAAAAAAAyO8QFgAAAABRogEAAAAAAOjuEBYAAAAAaAQAAAwAAADI7xAWAAAAAFGiAQAA"
+			"AAAACO8QFgAAAABpBAAAAAAAAMjvEBYAAAAAUaIBAAAAAAAo7xAWAAAAAGoEAAAAAAAAyO8QFgAA"
+			"AABRogEAAAAAAEjvEBYAAAAAawQAAAAAAADI7xAWAAAAAFGiAQAAAAAAaO8QFgAAAABvBAAAAAAA"
+			"AMjvEBYAAAAAUaIBAAAAAACI7xAWAAAAABgAAAAWfwAAIOsvDxd/AAABAAAAAAAAAEABERYAAAAA"
+			"+08AADcAAAD7TwAAOwAAABgAAAAAAAAAIOsvDxd/AAABAAAAAAAAAAUAAAAAAAAA+08AADcAAAD7"
+			"TwAAOwAAAG4EAAAAAAAAyO8QFgAAAABRogEAAAAAAKjvEBYAAAAAbAQAAGVnYTLI7xAWAAAAAFGi"
+			"AQAAAAAAKPAQFgAAAABZBAAAFgAAAAAAAAAAAAAAAAAAAAAAAAAAAAAAAAAAAAAAAAAAAAAAAAAA"
+			"AAAAAAAAAAAAAAAAAAAAAAAAAAAAAAAAAAAAAAAAAAAAAAAAAAAAAAAAAAAAAAAAAAAAAAAAAAAA"
+			"AAAAAAAAAAAAAAAAAAAAAAAAAAAAAAAAAAAAAAAAAAAAAAAAAAAAAAAAAAAAAAAAAAAAAAAAAAAA"
+			"AAAAAAAAAAAAAAAAAAAAAAAAAAAAAAAAAAAAAAAAAAAAAAAAAAAAAAAAAAAAAAAAAAAAAAAAAAAA"
+			"AAAAAAAAAAAAAAAAAAAAAAAAAAAAAAAAAAAAAAAAAAAAAAAAAAAAAAAAAAAAAAAAAAAAAAAAAAAA"
+			"AAAAAAAAAAAAAAAAAAAAAAAAAAAAAAAAAAAAAAAAAAAAAAAAAAAAAAAAAAAAAAAAAAAAAAAAAAAA"
+			"AAAAAAAAAAAAAAAAAAAAAAAAAAAAAAAAAAAAAAAAAAAAAAAAAAAAAAAAAAAAAAAAAAAAAAAAAAAA"
+			"AAAAAAAAAAAAAAAAAAAAAAAAAAAAAAAAAAAAAAAAAAAAAAAAAAAAAAAAAAAAAAAAAAAAAAAAAAAA"
+			"AAAAAAAAAAAAAAAAAAAAAAAAAAAAAAAAAAAAAAAAAAAAAAAAAAAAAAAAAAAAAAAAAAAAAAAAAAAA"
+			"AAAAAAAAAAAAAAAAAAAAAAAAAAAAAAAAAAAAAAAAAAAAAAAAAAAAAAAAAAAAAAAAAAAAAAAAAAAA"
+			"AAAAAAAAAAAAAAAAAAAAAAAAAAAAAAAAAAAAAAAAAAAAAAAAAAAAAAAAAAAAAAAAAAAAAAAAAAAA"
+			"AAAAAAAAAAAAAAAAAAAAAAAAAAAAAAAAAAAAAAAAAAAAAAAAAAAAAAAAAAAAAAAAAAAAAAAAAAAA"
+			"AAAAAAAAAAAAAAAAAAAAAAAAAAAAAAAAAAAAAAAAAAAAAAAAAAAAAAAAAAAAAAAAAAAAAAAAAAAA"
+			"AAAAAAAAAAAAAAAAAAAAAAAAAAAAAAAAAAAAAAAAAAAAAAAAAAAAAAAAAAAAAAAAAAAAAAAAAAAA"
+			"AAAAAAAAAAAAAAAAAAAAAAAAAAAAAAAAAAAAAAAAAAAAAAAAAAAAAAAAAAAAAAAAAAAAAAAAAAAA"
+			"AAAAAAAAAAAAAAAAAAAAAAAAAAAAAAAAAAAAAAAAAAAAAAAAAAAAAAAAAAAAAAAAAAAAAAAAAAAA"
+			"AAAAAAAAAAAAAAAAAAAAAAAAAAAAAAAAAAAAAAAAAAAAAAAAAAAAAAAAAAAAAAAAAAAAAAAAAAAA"
+			"AAAAAAAAAAAAAAAAAAAAAAAAAAAAAAAAAAAAAAAAAAAAAAAAAAAAAAAAAAAAAAAAAAAAAAAAAAAA"
+			"AAAAAAAAAAAAAAAAAAAAAAAAAA=="
 		)
 	)

Commit message: Novi raspored.
Parts:
- removed J12: Conn_01x04_Socket, Connector_JST:JST_PH_B4B-PH-K_1x04_P2.00mm_Vertical
- removed J6, J7: Wire2Board, Connector_Wire:SolderWire-0.127sqmm_1x01_D0.48mm_OD1mm
- removed Q2: FS8205A, Package_SO:TSSOP-8_4.4x3mm_P0.65mm
- removed R19: 0.4, Resistor_SMD:R_0603_1608Metric_Pad0.98x0.95mm_HandSolder
- removed R21: 10k, Resistor_SMD:R_0603_1608Metric_Pad0.98x0.95mm_HandSolder
- removed U2: TP4056, Package_SO:SOIC-8-1EP_3.9x4.9mm_P1.27mm_EP2.41x3.81mm
- added BT1: Battery_Cell, DS100M08KV:battery_holder, B.Cu at (140.0, 124.7)
- added D6: LED, LED_THT:LED_D3.0mm_FlatTop, F.Cu at (118.0, 141.1)
- added J2: Conn_01x04_Socket, Connector_JST:JST_PH_B4B-PH-K_1x04_P2.00mm_Vertical, B.Cu at (128.5, 141.1)
- added Q3: CMSN3416K-HF, Package_TO_SOT_SMD:SOT-23, F.Cu at (133.2, 145.4)
- added Q5: CMSN3416K-HF, Package_TO_SOT_SMD:SOT-23, F.Cu at (133.2, 148.9)
- added R36: 10k, Resistor_SMD:R_0603_1608Metric_Pad0.98x0.95mm_HandSolder, F.Cu at (121.3, 146.1)
- added U6: BQ21040DBV, Package_TO_SOT_SMD:SOT-23-6, F.Cu at (122.2, 142.1)
- C29, C3, RV2: moved to F.Cu
- H1, H2, H3, H4: footprint MountingHole:MountingHole_3.2mm_M3 -> DS100M08KV:M3_with_screw; moved to B.Cu
- J8: footprint DS100M08KV:red_safety_4mm_connector -> DS100M08KV:black_safety_4mm_connector
- Q1, Q4: footprint Package_TO_SOT_THT:TO-126-3_Horizontal_TabUp -> DS100M08KV:TO-126-3_Horizontal_TabUp_No_Hole
- R25: value 2k -> 10k
- R26: value 20k -> 330
- U5: value DW01A -> AP9101CAK6-ALTRG1
- moved C36 34.1 mm to (170.7, 141.2), turned to 0 degrees
- moved PS1 34.0 mm to (154.3, 149.1), turned to -90 degrees
- moved C40 31.1 mm to (138.3, 146.0), turned to -90 degrees
- moved R26 29.9 mm to (118.0, 145.8), turned to 0 degrees
- moved C28 29.0 mm to (155.5, 146.6), turned to 0 degrees
- moved R25 25.7 mm to (124.9, 142.1), turned to 90 degrees
- moved TP4 25.6 mm to (175.1, 136.9)
- moved C30 23.4 mm to (172.8, 134.4)
- moved RV4 22.6 mm to (148.7, 103.2)
- moved C20 21.6 mm to (166.9, 141.2), turned to 180 degrees
- moved Q1 18.3 mm to (153.7, 137.0), turned to 0 degrees
- moved C16 17.8 mm to (152.0, 141.2), turned to 0 degrees
- moved R30 17.5 mm to (124.3, 145.3), turned to 0 degrees
- moved Q4 17.2 mm to (166.5, 137.0), turned to 0 degrees
- moved C1 16.9 mm to (124.2, 139.1), turned to 180 degrees
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Connections:
- R26 pad 1: Earth -> Net-(D6-A)
- R26 pad 2: Net-(U2-TEMP) -> +VBUS
Routing:
- net +5V: track 137.4 -> 4.05 mm, vias 4 -> 3
- net -5V: track 119.8 -> 3.25 mm, vias 6 -> 4
- net Net-(PS1-+Vin): track 49.8 -> 0.00 mm
- net Net-(SW2A-B): track 41.0 -> 0.00 mm, vias 1 -> 0
- net +BAT: track 20.8 -> 0.00 mm, vias 1 -> 0
- net +VBUS: track 20.3 -> 0.00 mm
- net Earth: track 18.8 -> 0.00 mm, vias 13 -> 0
- net Net-(PS1-+Vout): track 17.3 -> 0.00 mm
- net Net-(PS1--Vout): track 12.4 -> 0.00 mm
- net Net-(U2-CE): track 11.5 -> 0.00 mm, vias 2 -> 0
- net 0: track 47.3 -> 39.4 mm, vias 25 -> 19
- net Net-(C4-Pad2): track 9.94 -> 2.13 mm
- net -BAT: track 7.27 -> 0.00 mm
- net Net-(SW1B-A): track 14.8 -> 21.0 mm
- net Net-(U5-CS): track 6.07 -> 0.00 mm
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- removed copper zone on In1.Cu, net 0
- removed copper zone on In1.Cu, net Earth
Other:
- board text removed: "+"
- board text removed: "-"

Commit message: Rutiranje.
Parts:
- removed U5: AP9101CAK6-ALTRG1, Package_TO_SOT_SMD:SOT-23-6
- added C45: 100n, Resistor_SMD:R_0603_1608Metric_Pad0.98x0.95mm_HandSolder, F.Cu at (137.8, 145.0)
- added U2: AP9101CK6, Package_TO_SOT_SMD:SOT-23-6, F.Cu at (143.4, 147.7)
- R29: value 1k -> 2.7k
- R30: value 100 -> 330
- moved R26 22.5 mm to (140.4, 144.1), turned to 90 degrees
- moved C1 22.3 mm to (146.5, 139.2), turned to 0 degrees
- moved C43 21.4 mm to (164.2, 141.1), turned to 90 degrees
- moved D6 17.5 mm to (133.8, 148.6), turned to 0 degrees
- moved C40 17.2 mm to (155.0, 150.1), turned to 90 degrees
- moved RV2 16.6 mm to (127.6, 123.6)
- moved C2 16.2 mm to (140.4, 149.1), turned to -90 degrees
- moved R33 16.2 mm to (179.6, 134.7), turned to 90 degrees
- moved BT1 16.0 mm to (156.0, 125.7)
- moved R5 15.7 mm to (125.6, 132.9), turned to -90 degrees
- moved R25 15.2 mm to (140.0, 140.0), turned to -90 degrees
- moved C41 15.2 mm to (163.8, 150.0)
- moved C42 15.2 mm to (163.8, 147.7)
- moved Q3 15.1 mm to (147.8, 149.3), turned to 90 degrees
- moved J11 15.1 mm to (178.3, 109.9)
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Routing:
- net -BAT: track 0.00 -> 67.4 mm, vias 0 -> 1
- net -5V: track 3.25 -> 67.8 mm
- net +5V: track 4.05 -> 62.3 mm
- net +BAT: track 0.00 -> 50.7 mm, vias 0 -> 3
- net Net-(PS1--Vout): track 0.00 -> 28.9 mm, vias 0 -> 1
- net Net-(PS1-+Vin): track 0.00 -> 25.1 mm, vias 0 -> 1
- net Net-(SW2A-B): track 0.00 -> 25.0 mm
- net Earth: track 0.00 -> 23.7 mm, vias 0 -> 9
- net Net-(PS1-+Vout): track 0.00 -> 22.2 mm
- net 0: track 39.4 -> 56.2 mm
- net Net-(C32-Pad2): track 2.11 -> 15.1 mm, vias 0 -> 1
- net Net-(D6-K): track 0.00 -> 9.98 mm
- net Net-(Q4-B): track 0.00 -> 9.74 mm
- net +VBUS: track 0.00 -> 8.85 mm, vias 0 -> 1
- net Net-(D6-A): track 0.00 -> 5.98 mm
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- added copper zone on In1.Cu, net 0
- added copper zone on In1.Cu, net Earth

Commit message: Rutiranje gotovo.
Parts:
- added J5: USB_C_floating, DS100M08KV:USB_C_floating, B.Cu at (203.3, 134.6)
- Q1, Q4: footprint DS100M08KV:TO-126-3_Horizontal_TabUp_No_Hole -> Package_TO_SOT_THT:TO-126-3_Vertical
- moved C29 10.3 mm to (177.8, 131.5), turned to 180 degrees
- moved J10 4.30 mm to (210.2, 114.0)
- moved FB4 2.88 mm to (174.5, 105.5), turned to 0 degrees
- moved R33 1.14 mm to (178.7, 134.0)
- moved R34 1.14 mm to (177.0, 134.0)
- moved R31 0.90 mm to (169.3, 134.7)
- moved R32 0.90 mm to (169.3, 133.1)
- moved C30 0.80 mm to (187.8, 134.6)
- moved C31 0.80 mm to (172.8, 134.7)
- moved J8 0.50 mm to (107.9, 138.0)
- moved H2 0.22 mm to (194.9, 108.5)
- moved H4 0.22 mm to (194.9, 143.5)
- moved H1 0.20 mm to (115.0, 108.5)
- moved H3 0.20 mm to (115.0, 143.5)
Routing:
- net +5V: track 62.3 -> 179.5 mm, vias 3 -> 2
- net -5V: track 67.8 -> 149.0 mm
- net Net-(C4-Pad2): track 2.13 -> 18.8 mm, vias 0 -> 1
- net 0: track 56.2 -> 62.3 mm, vias 19 -> 24
- net Net-(Q1-B): track 4.90 -> 9.93 mm
- net +BAT: track 50.7 -> 54.1 mm, vias 3 -> 2
- net Net-(PS1-+Vout): track 22.2 -> 25.3 mm
- net Net-(C11-Pad1): track 21.3 -> 24.2 mm
- net Net-(C15-Pad1): track 15.1 -> 18.0 mm
- net Earth: track 23.7 -> 26.6 mm
- net +VBUS: track 8.85 -> 11.2 mm, vias 1 -> 0
- net Net-(PS1--Vout): track 28.9 -> 26.7 mm
- net Net-(Q4-B): track 9.74 -> 11.4 mm
- net -BAT: track 67.4 -> 68.7 mm

Commit message: README.
Parts:
- moved RV4 1.73 mm to (162.2, 105.0)
Routing:
- net +5V: track 179.5 -> 181.9 mm
- net Net-(C4-Pad2): track 18.8 -> 16.7 mm
- net -5V: track 149.0 -> 148.2 mm
Changed lines of the file:
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@@
 	(footprint "Potentiometer_THT:Potentiometer_Bourns_3296W_Vertical"
 		(layer "B.Cu")
-		(at 163.72375 104.17375)
+		(at 162.2 105)
 		(descr "Potentiometer, vertical, Bourns 3296W, https://www.bourns.com/pdfs/3296.pdf")
 		(tags "Potentiometer vertical Bourns 3296W")
@@
 	)
 	(segment
+		(start 157.1 101.6)
+		(end 157.1 104.98)
+		(width 1)
+		(layer "F.Cu")
+		(net 6)
+	)
+	(segment
 		(start 173.7125 137.5475)
 		(end 173.26 138)
@@
 	)
 	(segment
-		(start 164.3 101.6)
-		(end 158.64375 101.6)
-		(width 1)
-		(layer "F.Cu")
-		(net 6)
-	)
-	(segment
 		(start 134.8625 122.95)
 		(end 134.8625 123.1375)
@@
 	)
 	(segment
+		(start 157.1 104.98)
+		(end 157.12 105)
+		(width 1)
+		(layer "F.Cu")
+		(net 6)
+	)
+	(segment
 		(start 175.375 105.075)
 		(end 171.9 101.6)
@@
 	)
 	(segment
-		(start 158.64375 101.6)
-		(end 158.64375 104.17375)
-		(width 1)
-		(layer "F.Cu")
-		(net 6)
-	)
-	(segment
 		(start 135.7 104.3)
 		(end 132.35 107.65)
@@
 	)
 	(segment
+		(start 164.3 101.6)
+		(end 157.1 101.6)
+		(width 1)
+		(layer "F.Cu")
+		(net 6)
+	)
+	(segment
 		(start 175.375 105.5)
 		(end 175.375 105.075)
@@
 	)
 	(segment
-		(start 163.72375 104.17375)
-		(end 162 105.8975)
+		(start 170.6 118)
+		(end 170.6 118.05705)
 		(width 1)
 		(layer "In2.Cu")
@@
 	)
 	(segment
-		(start 170.6 118)
-		(end 170.6 118.05705)
+		(start 161.3 113.6)
+		(end 163.6 115.9)
 		(width 1)
 		(layer "In2.Cu")
@@
 	)
 	(segment
+		(start 170.6 117.7)
+		(end 170.6 118)
+		(width 1)
+		(layer "In2.Cu")
+		(net 7)
+	)
+	(segment
 		(start 131.042521 141.2)
 		(end 132.903496 141.2)
@@
 	)
 	(segment
-		(start 170.6 117.7)
-		(end 170.6 118)
-		(width 1)
-		(layer "In2.Cu")
-		(net 7)
-	)
-	(segment
 		(start 132.903496 141.2)
 		(end 135.1 139.003496)
@@
 	)
 	(segment
+		(start 168.8 115.9)
+		(end 170.6 117.7)
+		(width 1)
+		(layer "In2.Cu")
+		(net 7)
+	)
+	(segment
 		(start 134 117.2)
 		(end 134.3 116.9)
@@
 	)
 	(segment
-		(start 162 105.8975)
-		(end 162 114.3)
+		(start 161.3 105.9)
+		(end 161.3 113.6)
 		(width 1)
 		(layer "In2.Cu")
@@
 	)
 	(segment
-		(start 168.8 115.9)
-		(end 170.6 117.7)
+		(start 162.3 105)
+		(end 162.2 105)
 		(width 1)
 		(layer "In2.Cu")
@@
 	)
 	(segment
-		(start 162 114.3)
-		(end 163.6 115.9)
-		(width 1)
-		(layer "In2.Cu")
-		(net 7)
-	)
-	(segment
 		(start 135.1 132)
 		(end 141.3 125.8)
@@
 	)
 	(segment
-		(start 141.3 125.7)
-		(end 136.7 121.1)
-		(width 0.5)
+		(start 163.6 115.9)
+		(end 168.8 115.9)
+		(width 1)
 		(layer "In2.Cu")
 		(net 7)
 	)
 	(segment
-		(start 163.6 115.9)
-		(end 168.8 115.9)
+		(start 162.2 105)
+		(end 161.3 105.9)
 		(width 1)
 		(layer "In2.Cu")
@@
 	)
 	(segment
+		(start 141.3 125.7)
+		(end 136.7 121.1)
+		(width 0.5)
+		(layer "In2.Cu")
+		(net 7)
+	)
+	(segment
 		(start 107.2 136.5)
 		(end 109.4 136.5)
@@
 	)
 	(segment
-		(start 163.5125 118.6)
-		(end 163.5 118.6)
-		(width 1)
-		(layer "In2.Cu")
-		(net 63)
-	)
-	(segment
-		(start 159.7 105.6)
-		(end 161.12625 104.17375)
+		(start 159.7 114.8)
+		(end 159.7 105.6)
 		(width 1)
 		(layer "In2.Cu")
@@
 	)
 	(segment
-		(start 161.12625 104.17375)
-		(end 161.18375 104.17375)
-		(width 1)
-		(layer "In2.Cu")
-		(net 63)
-	)
-	(segment
-		(start 159.7 114.8)
-		(end 159.7 105.6)
+		(start 163.5125 118.6)
+		(end 163.5 118.6)
 		(width 1)
 		(layer "In2.Cu")
