File: DS100M08KV.kicad_pcb (KiCad board)
At the start: 4 copper layers, 100 x 52 mm, 129 parts, among them J1 wire2board, J10 BNC_panel_mount, J11 wire2board, J2 Conn_01x04_Socket, J3 wire2board, J4 wire2board, J5 USB_C_floating, J8 red_safety_4mm_connector, J9 black_safety_4mm_connector, Q1 BD679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

Commit message: Rounded traces..
Routing:
- net -5V: track 148.2 -> 146.0 mm
- net -BAT: track 68.7 -> 67.8 mm
- net Net-(SW2A-B): track 25.0 -> 24.2 mm
- net Net-(SW1A-C): track 19.5 -> 18.8 mm
- net Net-(PS1-+Vout): track 25.3 -> 24.7 mm
- net +BAT: track 54.1 -> 53.5 mm
- net Net-(C32-Pad2): track 15.1 -> 14.6 mm
- net Net-(SW1B-A): track 21.0 -> 20.5 mm

Commit message: Minor changes to schematic and PCB.
Parts:
- removed H3: MountingHole, DS100M08KV:M3_with_screw
- added TP5: TestPoint, TestPoint:TestPoint_Pad_D2.0mm, F.Cu at (131.8, 128.2)
- R13: value 500 -> 50
- R16: value 50 -> 10
- R20: value 500 -> 100
- R22: value 1k -> 200
- R28: value 10k -> 91k
- R32, R34: value 3k3 -> 2k2
- R6: value 50 -> 500
- U1: value AD8039 -> AD8066
Connections:
- net Net-(PS1-+Vin) renamed +5V_BOOST
Routing:
- net 0: track 62.1 -> 67.2 mm
