File: DS100M08KV.kicad_sch (KiCad schematic)
At the start: 144 parts, among them J1 wire2board, J10 BNC_panel_mount, J11 wire2board, J2 Wire2Board, J3 wire2board, J4 wire2board, J5 Wire2Board, J6 Wire2Board, J7 Wire2Board, J8 red_safety_4mm_connector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

Commit message: Cleaning up libraries.
Parts:
- removed H10, H11, H12, H13, H14, H15, H16, H17, H18, H19, H20, H9: MountingHole, MountingHole:MountingHole_3.2mm_M3, symbol Mechanical:MountingHole
- removed J10: BNC_panel_mount, DS100M06V_linear:BNC_panel_mount, symbol DS100M06V_linear:BNC_panel_mount
- removed J8: red_safety_4mm_connector, DS100M06V_linear:red_safety_4mm_connector, symbol DS100M06V_linear:red_safety_4mm_connector
- removed J9: black_safety_4mm_connector, DS100M06V_linear:red_safety_4mm_connector, symbol DS100M06V_linear:black_safety_4mm_connector
- added J10: BNC_panel_mount, DS100M08KV:BNC_panel_mount, symbol DS100M08KV:BNC_panel_mount
- added J8: red_safety_4mm_connector, DS100M08KV:red_safety_4mm_connector, symbol DS100M08KV:red_safety_4mm_connector
- added J9: black_safety_4mm_connector, DS100M08KV:black_safety_4mm_connector, symbol diff-probe:black_safety_4mm_connector
- SW1, SW2: footprint DS100M06V_linear:DPDT_bigger -> DS100M08KV:DPDT_bigger

Commit message: Housekeeping.
Parts:
- removed H5, H6, H7, H8: WireFeedHole, MountingHole:MountingHole_2.2mm_M2_ISO7380, symbol Mechanical:MountingHole
- removed L1: 4.7u, Inductor_SMD:L_Bourns_SRN6045TA, symbol solar_push_pull_sym_lib:SRN6045HA-4R7Y
- removed PS1: IA0509S, Converter_DCDC:Converter_DCDC_XP_POWER-IAxxxxS_THT, symbol all_symbols_used:IA0509S
- removed Q2: FS8205A, Package_SO:TSSOP-8_4.4x3mm_P0.65mm, symbol DS100M06V_linear:FS8205A
- removed U1: AD8039, Package_SO:SOIC-8_3.9x4.9mm_P1.27mm, symbol diff-probe:AD8039
- removed U2: TP4056, Package_SO:SOIC-8-1EP_3.9x4.9mm_P1.27mm_EP2.41x3.81mm, symbol DS100M06V_linear:TP4056
- removed U4: AD8009, Package_SO:SOIC-8_3.9x4.9mm_P1.27mm, symbol diff-probe:AD8009
- removed U5: DW01A, Package_TO_SOT_SMD:SOT-23-6, symbol DS100M06V_linear:DW01A
- removed U7: TLV61070ADBVR, Package_TO_SOT_SMD:SOT-23-6, symbol DS100M06V_linear:TLV61070ADBVR
- added L3: 4.7u, Inductor_SMD:L_Bourns_SRN6045TA, symbol Device:L
- added PS1: IA0509S, Converter_DCDC:Converter_DCDC_XP_POWER-IAxxxxS_THT, symbol Converter_DCDC:IA0509S
- added Q2: FS8205A, Package_SO:TSSOP-8_4.4x3mm_P0.65mm, symbol DS100M08KV:FS8205A
- added U1: AD8039, Package_SO:SOIC-8_3.9x4.9mm_P1.27mm, symbol DS100M08KV:AD8039
- added U2: TP4056, Package_SO:SOIC-8-1EP_3.9x4.9mm_P1.27mm_EP2.41x3.81mm, symbol DS100M08KV:TP4056
- added U4: AD8009, Package_SO:SOIC-8_3.9x4.9mm_P1.27mm, symbol DS100M08KV:AD8009
- added U5: DW01A, Package_TO_SOT_SMD:SOT-23-6, symbol DS100M08KV:DW01A
- added U7: TLV61070ADBVR, Package_TO_SOT_SMD:SOT-23-6, symbol DS100M08KV:TLV61070ADBVR
Connections:
- net +BAT: now also U2.5 (Bat)
- net -BAT: now also Q2.6 (S), Q2.7 (S)
- net 0: now also PS1.5 (0V)
- net Earth: now also PS1.2 (-Vin), Q2.2 (S), Q2.3 (S), U2.3 (GND), U2.9 (GND), U5.6 (GND), U7.2 (GND)
- net at C2.1, R30.2: now also U5.5 (VCC)
- net at C22.2, C25.2, C38.2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: now also U4.4 (V-)
- net at R29.2: now also U5.2 (CS), U5.4 (TD)
- net at C3.1, Q1.2 (C), R31.2: now also PS1.6 (+Vout)
- net at R13.1, R18.1, R6.1: now also U4.2 (-)
- net at R16.2, R20.2, R22.1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: now also U4.3 (+)
- net at R17.2, R18.2, R35.1: now also U4.6
- net at C21.2, C26.2, C37.2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: now also U4.7 (V+)
- net at C43.2, L2.1, SW2.2 (B): now also L3.1, U7.3 (EN), U7.6 (VI)
- net at L2.2: now also L3.2, U7.1 (SW)
- net at C17.2, C28.1, C40.1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: now also PS1.1 (+Vin), U7.5 (VOUT)
- net at C18.2, C27.2, C35.2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: now also U1.4 (V-)
- net at R27.2, R28.1: now also U7.4 (FB)
- net at SW1.2 (B): now also U1.1, U1.2 (-)
- net at D7.3 (K), R51.1: now also U1.3 (+)
- net at C19.2, C33.2, C34.2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: now also U1.8 (V+)
- net at R21.1, R26.2: now also U2.1 (TEMP)
- net at R25.2: now also U2.2 (PROG)
- net at R19.2: now also U2.4 (Vin), U2.8 (CE)
- net at SW1.5 (B): now also U1.6 (-), U1.7
- net at C29.1, Q4.2 (C), R33.2: now also PS1.4 (-Vout)
- net at D2.3 (K), R52.1: now also U1.5 (+)
- new net: Q2.4 (G), U5.3 (OC)
- new net: Q2.5 (G), U5.1 (OD)
- no-connect marks 0 -> 2

Commit message: Clearer
Parts:
- removed J2, J5: Wire2Board, Connector_Wire:SolderWire-0.127sqmm_1x01_D0.48mm_OD1mm, symbol Connectors_and_wire_to_board:Wire2Board
- added J12: Conn_01x04_Socket, Connector_JST:JST_PH_B4B-PH-K_1x04_P2.00mm_Vertical, symbol Connector:Conn_01x04_Socket
Connections:
- net +VBUS: now also J12.1 (Pin_1)
- net Earth: now also J12.4 (Pin_4)
- no-connect marks 2 -> 4
Changed lines of the file:
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@@
 	)
 	(no_connect
+		(at 26.67 247.65)
+	)
+	(no_connect
+		(at 26.67 250.19)
+	)
+	(no_connect
 		(at 90.17 256.54)
 	)
 	(wire
 		(pts
-			(xy 34.29 257.81) (xy 35.56 257.81)
+			(xy 26.67 257.81) (xy 35.56 257.81)
 		)
 		(stroke
@@
 	(wire
 		(pts
-			(xy 46.99 257.81) (xy 46.99 260.35)
+			(xy 35.56 257.81) (xy 35.56 260.35)
+		)
+		(stroke
+			(width 0)
+			(type default)
+		)
+	)
+	(wire
+		(pts
+			(xy 26.67 245.11) (xy 26.67 240.03)
 		)
 		(stroke
@@
 	(wire
 		(pts
+			(xy 26.67 252.73) (xy 26.67 257.81)
+		)
+		(stroke
+			(width 0)
+			(type default)
+		)
+	)
+	(wire
+		(pts
 			(xy 367.03 107.95) (xy 378.46 107.95)
 		)
@@
 	(wire
 		(pts
+			(xy 26.67 240.03) (xy 35.56 240.03)
+		)
+		(stroke
+			(width 0)
+			(type default)
+		)
+	)
+	(wire
+		(pts
 			(xy 328.93 85.09) (xy 335.28 85.09)
 		)
@@
 	(wire
 		(pts
-			(xy 35.56 257.81) (xy 46.99 257.81)
-		)
-		(stroke
-			(width 0)
-			(type default)
-		)
-	)
-	(wire
-		(pts
 			(xy 331.47 40.64) (xy 322.58 40.64)
 		)
@@
 	(wire
 		(pts
-			(xy 35.56 240.03) (xy 44.45 240.03)
+			(xy 35.56 240.03) (xy 39.37 240.03)
 		)
 		(stroke
@@
 	(wire
 		(pts
-			(xy 34.29 240.03) (xy 35.56 240.03)
-		)
-		(stroke
-			(width 0)
-			(type default)
-		)
-	)
-	(wire
-		(pts
 			(xy 321.31 85.09) (xy 328.93 85.09)
 		)
@@
 	)
 	(global_label "+VBUS"
-		(shape input)
-		(at 44.45 240.03 0)
+		(shape output)
+		(at 39.37 240.03 0)
 		(fields_autoplaced yes)
 		(effects
@@
 		)
 		(property "Intersheetrefs" "${INTERSHEET_REFS}"
-			(at 53.9062 240.03 0)
+			(at 48.8262 240.03 0)
 			(effects
 				(font
@@
 	(symbol
 		(lib_id "power:Earth")
-		(at 46.99 260.35 0)
+		(at 35.56 260.35 0)
 		(unit 1)
 		(exclude_from_sim no)
@@
 		(fields_autoplaced yes)
 		(property "Reference" "#PWR07"
-			(at 46.99 266.7 0)
+			(at 35.56 266.7 0)
 			(effects
 				(font
@@
 		)
 		(property "Value" "Earth"
-			(at 46.99 265.43 0)
+			(at 35.56 265.43 0)
 			(effects
 				(font
@@
 		)
 		(property "Footprint" ""
-			(at 46.99 260.35 0)
+			(at 35.56 260.35 0)
 			(effects
 				(font
@@
 		)
 		(property "Datasheet" "~"
-			(at 46.99 260.35 0)
+			(at 35.56 260.35 0)
 			(effects
 				(font
@@
 		)
 		(property "Description" "Power symbol creates a global label with name \"Earth\""
-			(at 46.99 260.35 0)
+			(at 35.56 260.35 0)
 			(effects
 				(font
@@
 			)
 		)
-		(property "Description" ""
+		(property "Description" "Switch, dual pole double throw, separate symbols"
 			(at 189.23 180.34 0)
 			(effects
@@
 	)
 	(symbol
-		(lib_id "Connectors_and_wire_to_board:Wire2Board")
-		(at 29.21 240.03 0)
-		(mirror y)
-		(unit 1)
-		(exclude_from_sim no)
-		(in_bom yes)
-		(on_board yes)
-		(dnp no)
-		(fields_autoplaced yes)
-		(property "Reference" "J2"
-			(at 29.21 233.68 0)
-			(effects
-				(font
-					(size 1.27 1.27)
-				)
-			)
-		)
-		(property "Value" "Wire2Board"
-			(at 29.21 236.22 0)
-			(effects
-				(font
-					(size 1.27 1.27)
-				)
-			)
-		)
-		(property "Footprint" "Connector_Wire:SolderWire-0.127sqmm_1x01_D0.48mm_OD1mm"
-			(at 29.21 240.03 0)
-			(effects
-				(font
-					(size 1.27 1.27)
-				)
-				(hide yes)
-			)
-		)
-		(property "Datasheet" "~"
-			(at 29.21 240.03 0)
-			(effects
-				(font
-					(size 1.27 1.27)
-				)
-				(hide yes)
-			)
-		)
-		(property "Description" ""
-			(at 29.21 240.03 0)
-			(effects
-				(font
-					(size 1.27 1.27)
-				)
-				(hide yes)
-			)
-		)
-		(pin "1"
-		)
-		(instances
-			(project "DS100M06V_linear"
-				(path "/e034a6c3-9973-4355-8043-c1e988e27610"
-					(reference "J2")
-					(unit 1)
-				)
-			)
-		)
-	)
-	(symbol
 		(lib_id "Device:R_Potentiometer")
 		(at 163.83 71.12 180)
@@
 	)
 	(symbol
+		(lib_id "Connector:Conn_01x04_Socket")
+		(at 21.59 247.65 0)
+		(mirror y)
+		(unit 1)
+		(exclude_from_sim no)
+		(in_bom yes)
+		(on_board yes)
+		(dnp no)
+		(property "Reference" "J12"
+			(at 18.288 248.666 0)
+			(effects
+				(font
+					(size 1.27 1.27)
+				)
+			)
+		)
+		(property "Value" "Conn_01x04_Socket"
+			(at 22.225 242.57 0)
+			(effects
+				(font
+					(size 1.27 1.27)
+				)
+				(hide yes)
+			)
+		)
+		(property "Footprint" "Connector_JST:JST_PH_B4B-PH-K_1x04_P2.00mm_Vertical"
+			(at 21.59 247.65 0)
+			(effects
+				(font
+					(size 1.27 1.27)
+				)
+				(hide yes)
+			)
+		)
+		(property "Datasheet" "~"
+			(at 21.59 247.65 0)
+			(effects
+				(font
+					(size 1.27 1.27)
+				)
+				(hide yes)
+			)
+		)
+		(property "Description" "Generic connector, single row, 01x04, script generated"
+			(at 21.59 247.65 0)
+			(effects
+				(font
+					(size 1.27 1.27)
+				)
+				(hide yes)
+			)
+		)
+		(pin "3"
+		)
+		(pin "4"
+		)
+		(pin "2"
+		)
+		(pin "1"
+		)
+		(instances
+			(project ""
+				(path "/e034a6c3-9973-4355-8043-c1e988e27610"
+					(reference "J12")
+					(unit 1)
+				)
+			)
+		)
+	)
+	(symbol
 		(lib_id "Simulation_SPICE:0")
 		(at 369.57 74.93 0)
@@
 					(unit 1)
 				)
-			)
-		)
-	)
-	(symbol
-		(lib_id "Connectors_and_wire_to_board:Wire2Board")
-		(at 29.21 257.81 0)
-		(mirror y)
-		(unit 1)
-		(exclude_from_sim no)
-		(in_bom yes)
-		(on_board yes)
-		(dnp no)
-		(fields_autoplaced yes)
-		(property "Reference" "J5"
-			(at 29.21 251.46 0)
-			(effects
-				(font
-					(size 1.27 1.27)
-				)
-			)
-		)
-		(property "Value" "Wire2Board"
-			(at 29.21 254 0)
-			(effects
-				(font
-					(size 1.27 1.27)
-				)
-			)
-		)
-		(property "Footprint" "Connector_Wire:SolderWire-0.127sqmm_1x01_D0.48mm_OD1mm"
-			(at 29.21 257.81 0)
-			(effects
-				(font
-					(size 1.27 1.27)
-				)
-				(hide yes)
-			)
-		)
-		(property "Datasheet" "~"
-			(at 29.21 257.81 0)
-			(effects
-				(font
-					(size 1.27 1.27)
-				)
-				(hide yes)
-			)
-		)
-		(property "Description" ""
-			(at 29.21 257.81 0)
-			(effects
-				(font
-					(size 1.27 1.27)
-				)
-				(hide yes)
-			)
-		)
-		(pin "1"
-		)
-		(instances
-			(project "DS100M06V_linear"
-				(path "/e034a6c3-9973-4355-8043-c1e988e27610"
-					(reference "J5")
-					(unit 1)
-				)

Commit message: small updates.
Parts:
- removed Q2: FS8205A, Package_SO:TSSOP-8_4.4x3mm_P0.65mm, symbol DS100M08KV:FS8205A
- removed R19: 0.4, Resistor_SMD:R_0603_1608Metric_Pad0.98x0.95mm_HandSolder, symbol Device:R
- removed R21: 10k, Resistor_SMD:R_0603_1608Metric_Pad0.98x0.95mm_HandSolder, symbol Device:R
- removed U2: TP4056, Package_SO:SOIC-8-1EP_3.9x4.9mm_P1.27mm_EP2.41x3.81mm, symbol DS100M08KV:TP4056
- removed U5: DW01A, Package_TO_SOT_SMD:SOT-23-6, symbol DS100M08KV:DW01A
- added D6: LED, LED_THT:LED_D3.0mm_FlatTop, symbol Device:LED
- added Q3, Q5: CMSN3416K-HF, Package_TO_SOT_SMD:SOT-23, symbol Transistor_FET:BSS123
- added R36: 10k, Resistor_SMD:R_0603_1608Metric_Pad0.98x0.95mm_HandSolder, symbol Device:R
- added U5: AP9101CAK6-ALTRG1, Package_TO_SOT_SMD:SOT-23-6, symbol DS100M08KV:AP9101CAK6-ALTRG1
- added U6: BQ21040DBV, Package_TO_SOT_SMD:SOT-23-6, symbol Battery_Management:BQ21040DBV
- R25: value 2k -> 10k
- R26: value 20k -> 330
Connections:
- net +BAT: now also U6.2 (OUT)
- net +VBUS: now also R26.2, U6.6 (VIN)
- net -BAT: now also Q5.2 (S)
- net Earth: now also Q3.2 (S), R36.1, U5.6 (GND), U6.5 (GND); no longer R26.1
- net at C2.1, R30.2: now also U5.5 (VCC)
- net at R25.2: now also U6.1 (TS)
- net at R29.2: now also U5.2 (CS), U5.4 (TD)
- new net: D6.2 (A), R26.1
- new net: D6.1 (K), U6.3 (~{CHG})
- new net: R36.2, U6.4 (ISET)
- new net: Q5.1 (G), U5.1 (OD)
- new net: Q3.1 (G), U5.3 (OC)
- new net: Q3.3 (D), Q5.3 (D)
- no-connect marks 4 -> 2
Other:
- note added: "CONSIDER MEZANINE BOTTOM BOARD for the battery"
- note added: "Move all trim pots inline"
- note added: "https://www.kupujemprodajem.com/elektronika-i-komponente/moduli-za-samoizgradnju/nosac-drzac-18650-3-6v-3-7v-li-ion-baterija-jedno-leziste/oglas/51991902?filterId=6639827329"
- moved on the sheet: J6, J7, R25

Commit message: Novi raspored.
Parts:
- removed J12: Conn_01x04_Socket, Connector_JST:JST_PH_B4B-PH-K_1x04_P2.00mm_Vertical, symbol Connector:Conn_01x04_Socket
- removed J6, J7: Wire2Board, Connector_Wire:SolderWire-0.127sqmm_1x01_D0.48mm_OD1mm, symbol Connectors_and_wire_to_board:Wire2Board
- added BT1: Battery_Cell, DS100M08KV:battery_holder, symbol Device:Battery_Cell
- added J2: Conn_01x04_Socket, Connector_JST:JST_PH_B4B-PH-K_1x04_P2.00mm_Vertical, symbol Connector:Conn_01x04_Socket
- H1, H2, H3, H4: footprint MountingHole:MountingHole_3.2mm_M3 -> DS100M08KV:M3_with_screw
- J8: footprint DS100M08KV:red_safety_4mm_connector -> DS100M08KV:black_safety_4mm_connector
- Q1, Q4: footprint Package_TO_SOT_THT:TO-126-3_Horizontal_TabUp -> DS100M08KV:TO-126-3_Horizontal_TabUp_No_Hole
Connections:
- net +BAT: now also BT1.1 (+)
- net +VBUS: now also J2.1 (Pin_1)
- net -BAT: now also BT1.2 (-)
- net Earth: now also J2.4 (Pin_4)

Commit message: Rutiranje.
Parts:
- removed U5: AP9101CAK6-ALTRG1, Package_TO_SOT_SMD:SOT-23-6, symbol DS100M08KV:AP9101CAK6-ALTRG1
- added C45: 100n, Resistor_SMD:R_0603_1608Metric_Pad0.98x0.95mm_HandSolder, symbol Device:C
- added U2: AP9101CK6, Package_TO_SOT_SMD:SOT-23-6, symbol Battery_Management:AP9101CK6
- R29: value 1k -> 2.7k
- R30: value 100 -> 330
Connections:
- net +VBUS: now also C45.1
- net Earth: now also C45.2, U2.6 (VSS)
- net at C2.1, R30.2: now also U2.5 (VDD)
- net at Q5.1 (G): now also U2.3 (CO)
- net at R29.2: now also U2.2 (VM)
- net at Q3.1 (G): now also U2.1 (DO)
Other:
- moved on the sheet: C2, R30

Commit message: Rutiranje gotovo.
Parts:
- added J5: USB_C_floating, DS100M08KV:USB_C_floating, symbol DS100M08KV:USB_C_floating
- Q1, Q4: footprint DS100M08KV:TO-126-3_Horizontal_TabUp_No_Hole -> Package_TO_SOT_THT:TO-126-3_Vertical
Other:
- moved on the sheet: C1, C2, J2, Q3, Q5, R29, R30, U2

Commit message: README.
Connections:
- net +5V_BOOST: now reaches C17.2, C28.1, C40.1, C41.2, C42.2, PS1.1 (+Vin), R28.2, U7.5 (VOUT)
Other:
- note removed: "CONSIDER MEZANINE BOTTOM BOARD for the battery"
- note removed: "Move all trim pots inline"
- note removed: "https://www.kupujemprodajem.com/elektronika-i-komponente/moduli-za-samoizgradnju/nosac-drzac-18650-3-6v-3-7v-li-ion-baterija-jedno-leziste/oglas/51991902?filterId=6639827329"
- moved on the sheet: BT1, C16, C17, C20, C28, C29, C3, C30, C31, C36, C40, C41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
