File: DS100M08KV.kicad_sch (KiCad schematic)
At the start: 129 parts, among them J1 wire2board, J10 BNC_panel_mount, J11 wire2board, J2 Conn_01x04_Socket, J3 wire2board, J4 wire2board, J5 USB_C_floating, J8 red_safety_4mm_connector, J9 black_safety_4mm_connector, Q1 BD679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

Commit message: Minor update
Other:
- title: 1:200 600V 100 MHz differential probe -> 1:200 800V 100 MHz differential probe
Changed lines of the file:
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@@
 	(paper "A3")
 	(title_block
-		(title "1:200 600V 100 MHz differential probe")
+		(title "1:200 800V 100 MHz differential probe")
 		(rev "v1")
 		(company "TPI")

Commit message: Minor changes to schematic and PCB.
Parts:
- removed H3: MountingHole, DS100M08KV:M3_with_screw, symbol Mechanical:MountingHole
- added TP5: TestPoint, TestPoint:TestPoint_Pad_D2.0mm, symbol Connector:TestPoint
- R13: value 500 -> 50
- R16: value 50 -> 10
- R20: value 500 -> 100
- R22: value 1k -> 200
- R28: value 10k -> 91k
- R32, R34: value 3k3 -> 2k2
- R6: value 50 -> 500
- U1: value AD8039 -> AD8066
Connections:
- net 0: now also TP5.1
Other:
- moved on the sheet: RV2
Changed lines of the file:
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@@
 	(wire
 		(pts
-			(xy 85.09 71.12) (xy 85.09 82.55)
+			(xy 85.09 71.12) (xy 85.09 91.44)
 		)
 		(stroke
@@
 	(wire
 		(pts
-			(xy 85.09 90.17) (xy 85.09 109.22)
-		)
-		(stroke
-			(width 0)
-			(type default)
-		)
-	)
-	(wire
-		(pts
 			(xy 129.54 265.43) (xy 129.54 266.7)
 		)
@@
 	(wire
 		(pts
+			(xy 104.14 91.44) (xy 104.14 95.25)
+		)
+		(stroke
+			(width 0)
+			(type default)
+		)
+	)
+	(wire
+		(pts
 			(xy 129.54 266.7) (xy 132.08 266.7)
 		)
@@
 	(wire
 		(pts
-			(xy 91.44 86.36) (xy 88.9 86.36)
+			(xy 41.91 196.85) (xy 41.91 204.47)
 		)
 		(stroke
@@
 	(wire
 		(pts
-			(xy 41.91 196.85) (xy 41.91 204.47)
+			(xy 278.13 40.64) (xy 278.13 43.18)
 		)
 		(stroke
@@
 	(wire
 		(pts
-			(xy 278.13 40.64) (xy 278.13 43.18)
+			(xy 269.24 74.93) (xy 256.54 74.93)
 		)
 		(stroke
@@
 	(wire
 		(pts
-			(xy 269.24 74.93) (xy 256.54 74.93)
+			(xy 88.9 95.25) (xy 95.25 95.25)
+		)
+		(stroke
+			(width 0)
+			(type default)
+		)
+	)
+	(wire
+		(pts
+			(xy 85.09 99.06) (xy 85.09 109.22)
 		)
 		(stroke
@@
 			)
 		)
-		(property "Value" "500"
+		(property "Value" "100"
 			(at 297.942 73.914 90)
 			(effects
@@
 			)
 		)
-		(property "Value" "3k3"
+		(property "Value" "2k2"
 			(at 356.87 236.2199 0)
 			(effects
@@
 			)
 		)
-		(property "Value" "3k3"
+		(property "Value" "2k2"
 			(at 356.87 200.6599 0)
 			(effects
@@
 		(fields_autoplaced yes)
 		(property "Reference" "R28"
-			(at 227.33 259.08 0)
+			(at 227.33 259.0799 0)
 			(effects
 				(font
@@
 			)
 		)
-		(property "Value" "10k"
-			(at 227.33 261.62 0)
+		(property "Value" "91k"
+			(at 227.33 261.6199 0)
 			(effects
 				(font
@@
 			)
 		)
-		(property "Value" "AD8039"
+		(property "Value" "AD8066"
 			(at 258.572 66.294 0)
 			(effects
@@
 			)
 		)
-		(property "Value" "500"
+		(property "Value" "50"
 			(at 295.91 118.11 90)
 			(effects
@@
 	(symbol
 		(lib_id "Connector:TestPoint")
+		(at 104.14 91.44 0)
+		(unit 1)
+		(exclude_from_sim no)
+		(in_bom yes)
+		(on_board yes)
+		(dnp no)
+		(fields_autoplaced yes)
+		(property "Reference" "TP5"
+			(at 106.68 86.868 0)
+			(effects
+				(font
+					(size 1.27 1.27)
+				)
+				(justify left)
+			)
+		)
+		(property "Value" "TestPoint"
+			(at 106.68 89.408 0)
+			(effects
+				(font
+					(size 1.27 1.27)
+				)
+				(justify left)
+			)
+		)
+		(property "Footprint" "TestPoint:TestPoint_Pad_D2.0mm"
+			(at 109.22 91.44 0)
+			(effects
+				(font
+					(size 1.27 1.27)
+				)
+				(hide yes)
+			)
+		)
+		(property "Datasheet" "~"
+			(at 109.22 91.44 0)
+			(effects
+				(font
+					(size 1.27 1.27)
+				)
+				(hide yes)
+			)
+		)
+		(property "Description" ""
+			(at 104.14 91.44 0)
+			(effects
+				(font
+					(size 1.27 1.27)
+				)
+				(hide yes)
+			)
+		)
+		(pin "1"
+		)
+		(instances
+			(project "DS100M08KV"
+				(path "/e034a6c3-9973-4355-8043-c1e988e27610"
+					(reference "TP5")
+					(unit 1)
+				)
+			)
+		)
+	)
+	(symbol
+		(lib_id "Connector:TestPoint")
 		(at 97.79 57.15 0)
 		(unit 1)
@@
 			)
 		)
-		(property "Value" "1k"
+		(property "Value" "200"
 			(at 318.77 68.58 90)
 			(effects
@@
 	(symbol
 		(lib_id "Device:R_Potentiometer")
-		(at 85.09 86.36 0)
+		(at 85.09 95.25 0)
 		(mirror x)
 		(unit 1)
@@
 		(fields_autoplaced yes)
 		(property "Reference" "RV2"
-			(at 82.55 85.0899 0)
+			(at 82.55 93.9799 0)
 			(effects
 				(font
@@
 		)
 		(property "Value" "100"
-			(at 82.55 87.6299 0)
+			(at 82.55 96.5199 0)
 			(effects
 				(font
@@
 		)
 		(property "Footprint" "Potentiometer_THT:Potentiometer_Bourns_3296W_Vertical"
-			(at 85.09 86.36 0)
+			(at 85.09 95.25 0)
 			(effects
 				(font
@@
 		)
 		(property "Datasheet" "~"
-			(at 85.09 86.36 0)
+			(at 85.09 95.25 0)
 			(effects
 				(font
@@
 		)
 		(property "Description" ""
-			(at 85.09 86.36 0)
+			(at 85.09 95.25 0)
 			(effects
 				(font
@@
 			)
 		)
-		(property "Value" "50"
+		(property "Value" "500"
 			(at 295.91 105.41 90)
 			(effects
@@
 			)
 		)
-		(property "Value" "AD8039"
+		(property "Value" "AD8066"
 			(at 262.89 126.238 0)
 			(effects
@@
 			)
 		)
-		(property "Value" "AD8039"
+		(property "Value" "AD8066"
 			(at 261.62 52.578 0)
 			(effects
@@
 	)
 	(symbol
-		(lib_id "Mechanical:MountingHole")
-		(at 27.94 151.13 0)
-		(unit 1)
-		(exclude_from_sim no)
-		(in_bom yes)
-		(on_board yes)
-		(dnp no)
-		(property "Reference" "H3"
-			(at 30.48 149.86 0)
-			(effects
-				(font
-					(size 1.27 1.27)
-				)
-				(justify left)
-			)
-		)
-		(property "Value" "MountingHole"
-			(at 30.48 152.4 0)
-			(effects
-				(font
-					(size 1.27 1.27)
-				)
-				(justify left)
-			)
-		)
-		(property "Footprint" "DS100M08KV:M3_with_screw"
-			(at 27.94 151.13 0)
-			(effects
-				(font
-					(size 1.27 1.27)
-				)
-				(hide yes)
-			)
-		)
-		(property "Datasheet" "~"
-			(at 27.94 151.13 0)
-			(effects
-				(font
-					(size 1.27 1.27)
-				)
-				(hide yes)
-			)
-		)
-		(property "Description" ""
-			(at 27.94 151.13 0)
-			(effects
-				(font
-					(size 1.27 1.27)
-				)
-				(hide yes)
-			)
-		)
-		(instances
-			(project "DS100M06V_linear"
-				(path "/e034a6c3-9973-4355-8043-c1e988e27610"
-					(reference "H3")
-					(unit 1)
-				)
-			)
-		)
-	)
-	(symbol
 		(lib_id "DS100M06V_linear:1SV324")
 		(at 123.19 76.2 270)
@@
 			)
 		)
-		(property "Value" "50"
+		(property "Value" "10"
 			(at 295.91 63.5 90)
 			(effects
@@
 	(symbol
 		(lib_id "Simulation_SPICE:0")
-		(at 91.44 86.36 90)
+		(at 95.25 95.25 90)
 		(unit 1)
 		(exclude_from_sim no)
@@
 		(fields_autoplaced yes)
 		(property "Reference" "#GND01"
-			(at 93.98 86.36 0)
+			(at 97.79 95.25 0)
 			(effects
 				(font
@@
 		)
 		(property "Value" "0"
-			(at 88.9 86.36 0)
+			(at 92.71 95.25 0)
 			(effects
 				(font
@@
 		)
 		(property "Footprint" ""
-			(at 91.44 86.36 0)
+			(at 95.25 95.25 0)
 			(effects
 				(font
@@
 		)
 		(property "Datasheet" "~"
-			(at 91.44 86.36 0)
+			(at 95.25 95.25 0)
 			(effects
 				(font
@@
 		)
 		(property "Description" ""
-			(at 91.44 86.36 0)
+			(at 95.25 95.25 0)
 			(effects
 				(font
@@
 					(unit 1)
 				)
+			)
+		)
+	)
+	(symbol
+		(lib_id "Simulation_SPICE:0")
+		(at 104.14 95.25 0)
+		(unit 1)
+		(exclude_from_sim no)
+		(in_bom yes)
+		(on_board yes)
+		(dnp no)
+		(fields_autoplaced yes)
+		(property "Reference" "#GND038"
+			(at 104.14 97.79 0)
+			(effects
+				(font
+					(size 1.27 1.27)
+				)
+				(hide yes)
+			)
+		)
+		(property "Value" "0"
+			(at 104.14 92.71 0)
+			(effects
+				(font
+					(size 1.27 1.27)
+				)
+				(hide yes)
+			)
+		)
+		(property "Footprint" ""
+			(at 104.14 95.25 0)
+			(effects
+				(font
+					(size 1.27 1.27)
+				)
+				(hide yes)
+			)
+		)
+		(property "Datasheet" "~"
+			(at 104.14 95.25 0)
+			(effects
+				(font
+					(size 1.27 1.27)
+				)
+				(hide yes)
+			)
+		)
+		(property "Description" ""
+			(at 104.14 95.25 0)
+			(effects
+				(font
+					(size 1.27 1.27)
+				)
+				(hide yes)
+			)
+		)
+		(pin "1"
+		)
+		(instances
+			(project "DS100M08KV"
+				(path "/e034a6c3-9973-4355-8043-c1e988e27610"
+					(reference "#GND038")
+					(unit 1)
+				)
